File: qmd_hw.kicad_pcb (KiCad board)
At the start: 2 copper layers, 60 x 175 mm, 264 parts, among them J201 USB4120-03-C, J202 B2B-PH-SM4-TB(LF)(SN), J203 Screw_Terminal_01x02, J204 X4621FVS-2x20-C43D65, J205 X4621WVS-2x20I-C40D64, J206 X4621FVS-2x20-C43D65, J207 X4621FVS-2x20-C43D65, J208 NC_Conn_02x03_Odd_Even, J209 JST_PH_B3B-PH-SM4-TB, J210 NC_Conn_01x07_Female, J301 Screw_Terminal_01x01, J302 Screw_Terminal_01x01, J303 Conn_01x05_MountingPin, J304 X4621WVS-2x20I-C40D64, J305 X4621FVS-2x20-C43D65, J306 Screw_Terminal_01x01, J307 Screw_Terminal_01x01, J309 Screw_Terminal_01x01, J401 Screw_Terminal_01x01, J402 Screw_Terminal_01x01, J403 Screw_Terminal_01x01, J404 X4621WVS-2x20I-C40D64, J405 Screw_Terminal_01x01, J406 Conn_01x05_MountingPin, J408 X4621WVS-2x20I-C40D64, J409 Screw_Terminal_01x01, Q201 CSD18540Q5B, Q202 CSD18540Q5B, Q301 HYG025N06LS1C2, Q302 HYG025N06LS1C2, Q303 HYG025N06LS1C2, Q304 HYG025N06LS1C2, Q305 HYG025N06LS1C2, Q306 HYG025N06LS1C2, Q307 HYG025N06LS1C2, Q308 HYG025N06LS1C2, Q309 HYG025N06LS1C2, Q310 HYG025N06LS1C2, Q311 HYG025N06LS1C2, Q312 HYG025N06LS1C2, Q401 HYG025N06LS1C2, Q402 HYG025N06LS1C2, Q403 HYG025N06LS1C2, Q404 HYG025N06LS1C2, Q405 HYG025N06LS1C2, Q406 HYG025N06LS1C2, Q407 HYG025N06LS1C2, Q408 HYG025N06LS1C2, Q409 HYG025N06LS1C2, Q410 HYG025N06LS1C2, Q411 HYG025N06LS1C2, Q412 HYG025N06LS1C2, SW201 SW_DIP_x02, U201 STM32F405RGTx, U202 TJA1050T, U203 LM5109BSD, U204 LM1117-3.3, U205 LP5907MFX-3.3, U301 DRV8301DCAR, U401 DRV8301DCAR, Y201 8MHz

Commit message: Update artwork for M0 board
Parts:
- NT303: value NetTie_2 -> Net-Tie_2; footprint qdrive_footprints:NetTie-2_SMD_Pad2.0mm -> NetTie:NetTie-2_SMD_Pad0.5mm; moved to B.Cu
- R209: value 10k -> 21k
- moved C319 38.5 mm to (175.5, 123.9), turned to 180 degrees
- moved R314 32.3 mm to (163.1, 155.4), turned to 0 degrees
- moved C301 31.6 mm to (175.5, 127.9)
- moved C304 21.9 mm to (194.4, 128.3)
- moved L301 20.5 mm to (210.4, 111.4), turned to 90 degrees
- moved D301 20.2 mm to (204.0, 112.2)
- moved C325 20.2 mm to (194.5, 125.0)
- moved R301 20.2 mm to (205.4, 142.4)
- moved C314 18.7 mm to (178.9, 129.9)
- moved R302 17.0 mm to (198.0, 142.5)
- moved C323 16.7 mm to (204.8, 106.3)
- moved R313 16.6 mm to (173.4, 142.6)
- moved C336 14.8 mm to (190.5, 125.5), turned to -90 degrees
- moved C322 14.5 mm to (193.2, 122.7), turned to 0 degrees
- moved R310 13.9 mm to (189.4, 142.3)
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Connections:
- C302 pad 2: GND1 -> PGND_M0
- C307 pad 1: GND1 -> PGND_M0
- C309 pad 1: GND1 -> PGND_M0
- C310 pad 1: GND1 -> PGND_M0
- C311 pad 2: GND1 -> PGND_M0
- C312 pad 2: GND1 -> PGND_M0
- C315 pad 2: GND1 -> PGND_M0
- C320 pad 2: GND1 -> PGND_M0
- C321 pad 2: GND1 -> PGND_M0
- C323 pad 2: GND1 -> PGND_M0
- C324 pad 2: GND1 -> PGND_M0
- C326 pad 2: GND1 -> PGND_M0
- C333 pad 2: GND1 -> PGND_M0
- C334 pad 2: GND1 -> PGND_M0
- C335 pad 2: GND1 -> PGND_M0
- C336 pad 1: M0_3V3A -> 3V3A
- C336 pad 2: GND1 -> PGND_M0
- D301 pad 2: GND1 -> PGND_M0
- J303 pad 5: GND1 -> PGND_M0
- J303 pad MP: GND1 -> PGND_M0
- J304 pad 33: M0_3V3A -> unconnected-(J304-Pin_33-Pad33)
- J304 pad 37: GND1 -> PGND_M0
- J304 pad 38: GND1 -> PGND_M0
- J304 pad 39: GND1 -> PGND_M0
- J304 pad 40: GND1 -> PGND_M0
- NT303 pad 1: GND1 -> /M0_board/M0_SL_A
- R303 pad 1: GND1 -> PGND_M0
- R304 pad 2: GND1 -> PGND_M0
- R305 pad 2: GND1 -> PGND_M0
- R307 pad 1: GND1 -> PGND_M0
- R323 pad 1: GND1 -> PGND_M0
- U301 pad 24: M0_3V3A -> 3V3A
- U301 pad 28: GND1 -> PGND_M0
- U301 pad 44: PGND_M0 -> /M0_board/M0_SL_A
- U301 pad 57: GND1 -> PGND_M0
Routing:
- net VPP_M0: track 47.1 -> 0.00 mm, vias 82 -> 63
- net /M0_board/M0_GL_C: track 7.33 -> 46.3 mm, vias 0 -> 2
- net Net-(D301-K): track 0.00 -> 34.8 mm, vias 0 -> 3
- net M0_3V3A: track 32.7 -> 0.00 mm, vias 1 -> 0
- net Net-(Q311-G): track 40.2 -> 9.63 mm, vias 2 -> 0
- net PGND_M0: track 45.4 -> 15.4 mm, vias 72 -> 63
- net Net-(Q301-G): track 39.5 -> 14.1 mm
- net /M0_board/M0_GH_A: track 7.28 -> 28.7 mm, vias 0 -> 2
- net /M0_board/M0_GH_C: track 7.47 -> 27.9 mm, vias 0 -> 2
- net Net-(Q303-G): track 34.6 -> 14.2 mm, vias 2 -> 1
- net Net-(Q309-G): track 34.5 -> 14.4 mm
- net /M0_board/M0_GL_A: track 7.19 -> 26.2 mm, vias 0 -> 2
- net /M0_board/M0_SL_A: track 0.00 -> 18.4 mm, vias 0 -> 1
- net /M0_board/M0_GL_B: track 7.64 -> 24.0 mm, vias 0 -> 2
- net /M0_board/M0_GH_B: track 7.64 -> 23.2 mm, vias 0 -> 2
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- added copper zone on In1.Cu, net PGND_M0
- removed copper zone on B.Cu, net GND1
- removed copper zone on F.Cu, net GND1
- removed copper zone on F.Cu, net Net-(D301-K)
Other:
- copper layers 2 -> 4
- board text added: "BLDC DRIVE REV3"

Commit message: Added layer 3
Parts:
- moved L301 1.50 mm to (208.9, 111.4)
- moved C323 0.82 mm to (205.0, 107.1)
- moved C317 0.60 mm to (186.9, 126.6)
- moved R305 0.50 mm to (200.3, 108.0)
- moved NT302 0.40 mm to (175.7, 135.2)
- moved R317 0.32 mm to (180.9, 108.1)
- moved C309 0.28 mm to (180.9, 106.0)
- moved C312 0.28 mm to (183.2, 106.0)
- moved R311 0.20 mm to (185.6, 142.3)
- moved C310 0.10 mm to (178.9, 107.5)
- turned D301 to 90 degrees
Routing:
- net Net-(D301-K): track 34.8 -> 31.5 mm
- net +5V: track 81.6 -> 79.4 mm
- net /M0_board/M0_SL_B: track 22.6 -> 23.8 mm, vias 22 -> 23
- net /M0_board/M0_SH_C: track 33.3 -> 32.4 mm
- net /M0_board/M0_SH_A: track 32.3 -> 31.5 mm
- net /M0_board/M0_SH_B: track 26.1 -> 25.4 mm
- net /M0_board/M0_SP2: track 18.9 -> 18.2 mm, vias 1 -> 2
- net /M0_board/M0_SL_A: track 18.4 -> 17.7 mm, vias 1 -> 2
- net Net-(U301-BST_B): track 5.61 -> 6.21 mm
- net /M0_board/M0_GL_C: track 46.3 -> 45.7 mm
- net /M0_board/M0_SN1: track 19.5 -> 18.9 mm, vias 1 -> 2
- net Net-(U301-RT_CLK): track 8.60 -> 9.10 mm
- net /M0_board/M0_SN2: track 19.8 -> 19.4 mm, vias 1 -> 2
- net /M0_board/M0_SL_C: track 30.0 -> 29.6 mm, vias 22 -> 23
- net /M0_board/M0_SP1: track 21.4 -> 21.0 mm, vias 1 -> 2
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- added copper zone on In2.Cu, net PGND_M0

Commit message: Updated route per BOOSTXL reference design
Parts:
- removed TP301, TP302: TestPoint, TestPoint:TestPoint_Pad_D1.5mm
- C307: footprint Capacitor_SMD:C_0402_1005Metric -> Capacitor_SMD:C_0603_1608Metric
- NT303: moved to F.Cu
- moved NT303 7.45 mm to (195.6, 142.6)
- moved C312 5.73 mm to (179.1, 110.0), turned to 180 degrees
- moved R317 5.00 mm to (176.1, 106.7), turned to 180 degrees
- moved C309 4.82 mm to (176.1, 105.6), turned to 180 degrees
- moved C306 4.80 mm to (186.6, 110.2)
- moved R318 3.77 mm to (176.1, 107.8), turned to 180 degrees
- moved C310 3.13 mm to (176.1, 108.9), turned to 180 degrees
- moved C307 2.66 mm to (188.0, 108.0)
- moved C311 2.44 mm to (179.1, 111.5), turned to 180 degrees
- moved R307 2.30 mm to (195.2, 108.3)
- moved R306 2.30 mm to (196.3, 108.3)
- moved R303 1.92 mm to (186.3, 107.1)
- moved C303 1.71 mm to (188.3, 135.2)
- moved C323 1.70 mm to (204.2, 108.6), turned to 90 degrees
- moved NT301 1.46 mm to (188.8, 136.6), turned to -90 degrees
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Routing:
- net /M0_board/M0B_TEMP: track 31.7 -> 17.9 mm
- net /M0_board/M0_SL_A: track 17.7 -> 25.2 mm
- net Net-(U301-SO2): track 3.75 -> 11.2 mm, vias 0 -> 2
- net Net-(U301-SO1): track 4.52 -> 11.1 mm, vias 0 -> 2
- net /M0_board/M0B_SO2: track 27.9 -> 21.7 mm
- net /M0_board/M0B_SO1: track 28.3 -> 22.4 mm
- net /M0_board/M0B_nCS: track 36.3 -> 40.8 mm, vias 1 -> 2
- net Net-(U301-CP1): track 8.17 -> 4.08 mm
- net Net-(U301-CP2): track 6.96 -> 2.91 mm
- net /M0_board/M0_SH_A: track 31.5 -> 35.4 mm
- net /M0_board/M0_GH_A: track 28.7 -> 32.2 mm
- net /M0_board/M0B_PWRGD: track 47.5 -> 44.3 mm
- net /M0_board/M0BnOCTW: track 44.4 -> 41.7 mm
- net 3V3A: track 78.0 -> 80.6 mm
- net /M0_board/M0B_CL: track 24.4 -> 26.9 mm
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- added copper zone on F.Cu, net (none)
- removed copper zone on F.Cu, net /M0_board/M0_SL_C
