File: qmd_hw.kicad_pcb (KiCad board)
At the start: 4 copper layers, 60 x 175 mm, 262 parts, among them J201 USB4120-03-C, J202 B2B-PH-SM4-TB(LF)(SN), J203 Screw_Terminal_01x02, J204 X4621FVS-2x20-C43D65, J205 X4621WVS-2x20I-C40D64, J206 X4621FVS-2x20-C43D65, J207 X4621FVS-2x20-C43D65, J208 NC_Conn_02x03_Odd_Even, J209 JST_PH_B3B-PH-SM4-TB, J210 NC_Conn_01x07_Female, J301 Screw_Terminal_01x01, J302 Screw_Terminal_01x01, J303 Conn_01x05_MountingPin, J304 X4621WVS-2x20I-C40D64, J305 X4621FVS-2x20-C43D65, J306 Screw_Terminal_01x01, J307 Screw_Terminal_01x01, J309 Screw_Terminal_01x01, J401 Screw_Terminal_01x01, J402 Screw_Terminal_01x01, J403 Screw_Terminal_01x01, J404 X4621WVS-2x20I-C40D64, J405 Screw_Terminal_01x01, J406 Conn_01x05_MountingPin, J408 X4621WVS-2x20I-C40D64, J409 Screw_Terminal_01x01, Q201 CSD18540Q5B, Q202 CSD18540Q5B, Q301 HYG025N06LS1C2, Q302 HYG025N06LS1C2, Q303 HYG025N06LS1C2, Q304 HYG025N06LS1C2, Q305 HYG025N06LS1C2, Q306 HYG025N06LS1C2, Q307 HYG025N06LS1C2, Q308 HYG025N06LS1C2, Q309 HYG025N06LS1C2, Q310 HYG025N06LS1C2, Q311 HYG025N06LS1C2, Q312 HYG025N06LS1C2, Q401 HYG025N06LS1C2, Q402 HYG025N06LS1C2, Q403 HYG025N06LS1C2, Q404 HYG025N06LS1C2, Q405 HYG025N06LS1C2, Q406 HYG025N06LS1C2, Q407 HYG025N06LS1C2, Q408 HYG025N06LS1C2, Q409 HYG025N06LS1C2, Q410 HYG025N06LS1C2, Q411 HYG025N06LS1C2, Q412 HYG025N06LS1C2, SW201 SW_DIP_x02, U201 STM32F405RGTx, U202 TJA1050T, U203 LM5109BSD, U204 LM1117-3.3, U205 LP5907MFX-3.3, U301 DRV8301DCAR, U401 DRV8301DCAR, Y201 8MHz

Commit message: Re-route
Parts:
- moved C318 2.30 mm to (183.3, 127.1)
- moved C305 1.17 mm to (173.9, 135.8)
- moved R315 1.12 mm to (171.9, 135.8)
- moved C317 0.92 mm to (186.7, 127.5)
- moved C314 0.73 mm to (178.2, 130.1)
- moved R313 0.70 mm to (172.7, 142.6)
- moved Q309 0.65 mm to (174.6, 146.5)
- moved Q310 0.65 mm to (174.6, 153.5)
- moved Q311 0.55 mm to (167.2, 146.5)
- moved Q312 0.55 mm to (167.2, 153.5)
- moved C316 0.51 mm to (189.0, 125.6)
- moved NT303 0.45 mm to (195.5, 142.1), turned to 0 degrees
- moved Q304 0.45 mm to (200.2, 153.5)
- moved C336 0.41 mm to (190.1, 125.6)
- moved D301 0.40 mm to (203.9, 113.0)
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Routing:
- net /M0_board/M0_SH_B: track 24.6 -> 28.2 mm, vias 2 -> 3
- net /M0_board/M0_SP2: track 17.2 -> 19.7 mm
- net Net-(U301-BST_C): track 3.81 -> 6.25 mm
- net /M0_board/M0_SN2: track 18.3 -> 19.7 mm
- net /M0_board/M0_GL_B: track 22.8 -> 21.5 mm
- net /M0_board/M0_SH_C: track 31.6 -> 32.8 mm
- net /M0_board/M0_SH_A: track 35.4 -> 36.5 mm
- net /M0_board/M0_SN1: track 17.8 -> 18.8 mm, vias 2 -> 1
- net /M0_board/M0_GH_C: track 26.6 -> 27.5 mm
- net 3V3A: track 80.6 -> 81.5 mm
- net Net-(U301-BST_B): track 5.46 -> 6.28 mm
- net /M0_board/M0_GL_A: track 25.9 -> 26.7 mm
- net /M0_board/M0_SL_A: track 25.2 -> 24.5 mm
- net /M0_board/M0_GH_A: track 32.2 -> 32.7 mm
- net /M0_board/M0_GH_B: track 22.0 -> 22.5 mm, vias 2 -> 0
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- added copper zone on F.Cu, net /M0_board/M0_SL_C
- removed copper zone on F.Cu, net (none)

Commit message: Fixed bugs and parts update
Parts:
- removed C221: 4.7uF 50V, Capacitor_SMD:C_0805_2012Metric
- removed NT403: NetTie_2, qdrive_footprints:NetTie-2_SMD_Pad2.0mm
- removed TP401, TP402: TestPoint, TestPoint:TestPoint_Pad_D1.5mm
- removed U205: LP5907MFX-3.3, Package_TO_SOT_SMD:SOT-23-5
- added C434: 0.1uF 50V, Capacitor_SMD:C_0402_1005Metric, F.Cu at (184.9, 196.9)
- added NT404: Net-Tie_2, NetTie:NetTie-2_SMD_Pad0.5mm, F.Cu at (162.8, 172.7)
- added R235: 0R, Resistor_SMD:R_0603_1608Metric, F.Cu at (189.1, 93.7)
- C201, C202, C203, C204, C205, C206, C207, C208, C209, C210, C211, C212, C213, C214, C215, C216, C217, C218, C219, C223, C224, C225, C226, C311, C312, C323, C324, C326, C333, C334, C335, C407, C411, C412, C421, C423, C424, C425, C426, C433: footprint Capacitor_SMD:C_0402_1005Metric -> Capacitor_SMD:C_0603_1608Metric
- R201, R202, R203, R204, R205, R206, R207, R208, R209, R210, R211, R212, R213, R214, R215, R216, R217, R218, R219, R220, R221, R222, R223, R224, R225, R226, R227, R228, R229, R230, R231, R232, R233, R234, R301, R302, R307, R309, R310, R311, R313, R314, R315, R319, R320, R321, R323, R401, R402, R407, R409, R410, R411, R413, R414, R415, R419, R420, R421, R423: footprint Resistor_SMD:R_0402_1005Metric -> Resistor_SMD:R_0603_1608Metric
- moved C404 36.8 mm to (176.7, 194.5), turned to -135 degrees
- moved C422 27.7 mm to (179.2, 197.0), turned to -135 degrees
- moved R201 26.9 mm to (189.5, 61.5)
- moved R402 24.4 mm to (164.7, 180.6)
- moved R413 18.4 mm to (205.2, 180.4)
- moved D401 18.3 mm to (171.1, 212.9), turned to -90 degrees
- moved R401 18.0 mm to (172.0, 180.6)
- moved C401 14.7 mm to (198.6, 194.7), turned to 180 degrees
- moved R411 14.6 mm to (184.8, 180.4)
- moved R414 14.4 mm to (200.0, 180.4)
- moved R410 14.1 mm to (188.2, 180.4)
- moved C433 9.46 mm to (195.3, 214.6), turned to -90 degrees
- moved C430 9.42 mm to (213.8, 190.4)
- moved R421 8.13 mm to (180.7, 215.1)
- moved R419 8.08 mm to (179.2, 215.1)
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Connections:
- C402 pad 1: GND2 -> PGND_M1
- C407 pad 2: GND2 -> PGND_M1
- C409 pad 1: GND2 -> PGND_M1
- C410 pad 1: GND2 -> PGND_M1
- C411 pad 2: GND2 -> PGND_M1
- C412 pad 2: GND2 -> PGND_M1
- C419 pad 2: GND2 -> PGND_M1
- C421 pad 2: GND2 -> PGND_M1
- C423 pad 2: GND2 -> PGND_M1
- C424 pad 1: GND2 -> PGND_M1
- C425 pad 1: GND2 -> PGND_M1
- C426 pad 1: GND2 -> PGND_M1
- C433 pad 1: M1_3V3A -> 3V3B
- C433 pad 2: GND2 -> PGND_M1
- D401 pad 2: GND2 -> PGND_M1
- J404 pad 37: GND2 -> PGND_M1
- J404 pad 38: GND2 -> PGND_M1
- J404 pad 39: GND2 -> PGND_M1
- J404 pad 40: GND2 -> PGND_M1
- J406 pad 5: GND2 -> PGND_M1
- J406 pad MP: GND2 -> PGND_M1
- R403 pad 1: GND2 -> PGND_M1
- R404 pad 2: GND2 -> PGND_M1
- R405 pad 2: GND2 -> PGND_M1
- R407 pad 1: GND2 -> PGND_M1
- R423 pad 1: GND2 -> PGND_M1
- U401 pad 24: M1_3V3A -> 3V3B
- U401 pad 28: GND2 -> PGND_M1
- U401 pad 44: PGND_M1 -> /M1_board/M1_SL_A
- U401 pad 57: GND2 -> PGND_M1
Routing:
- net +5VA: track 151.6 -> 95.4 mm
- net M1_3V3A: track 52.9 -> 0.00 mm, vias 1 -> 0
- net /M1_board/M1_SL_A: track 0.00 -> 43.5 mm, vias 0 -> 2
- net VPP_M1: track 40.1 -> 0.00 mm, vias 53 -> 107
- net 3V3B: track 60.1 -> 96.4 mm, vias 1 -> 5
- net PGND_M1: track 49.2 -> 14.4 mm, vias 91 -> 276
- net Net-(Q403-G): track 40.2 -> 10.3 mm, vias 2 -> 0
- net /M1_board/M1_GL_A: track 6.10 -> 35.6 mm, vias 0 -> 2
- net +3.3VA: track 67.6 -> 38.5 mm, vias 4 -> 2
- net /main_board/M0_SO1: track 62.4 -> 39.0 mm, vias 0 -> 2
- net Net-(Q409-G): track 32.6 -> 9.77 mm
- net Net-(Q407-G): track 34.5 -> 12.3 mm, vias 2 -> 0
- net /M1_board/M1_GH_A: track 6.24 -> 28.1 mm, vias 0 -> 2
- net Net-(Q401-G): track 31.6 -> 9.91 mm
- net /M1_board/M1_GH_C: track 7.04 -> 28.2 mm, vias 0 -> 2
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- added copper zone on B.Cu, net /main_board/BRAKE_OUT
- added copper zone on In1.Cu, net GND
- added copper zone on In2.Cu, net GND
- added copper zone on In1.Cu, net PGND_M1
- added copper zone on In2.Cu, net PGND_M1
- removed copper zone on B.Cu, net GND2
- removed copper zone on F.Cu, net GND2
Other:
- board text added: "QDRIVE REV3 20230625"
- board text added: "V+"
- board text removed: "BLDC DRIVE REV2"
- board text removed: "QDRIVE REV2 20230419"

Commit message: Updated MB
Parts:
- removed J202: B2B-PH-SM4-TB(LF)(SN), Connector_JST:JST_PH_B2B-PH-SM4-TB_1x02-1MP_P2.00mm_Vertical
- added C221: 0.1uF 50V, Capacitor_SMD:C_0603_1608Metric, F.Cu at (180.6, 66.3)
- added C227: 1uF 35V, Capacitor_SMD:C_0603_1608Metric, F.Cu at (186.6, 68.7)
- added J211: S3B-PH-SM4-TB(LF)(SN), qdrive_footprints:JST_S3B-PH-SM4-TB, B.Cu at (196.4, 53.1)
- added JP207: Jumper_2_Open, Jumper:SolderJumper-2_P1.3mm_Open_TrianglePad1.0x1.5mm, B.Cu at (184.8, 49.2)
- added Q203: CSD18540Q5B, Package_TO_SOT_SMD:TDSON-8-1, B.Cu at (197.9, 66.9)
- added Q204: CSD18540Q5B, Package_TO_SOT_SMD:TDSON-8-1, F.Cu at (204.7, 66.2)
- added R236: 0R, Resistor_SMD:R_0603_1608Metric, F.Cu at (189.0, 92.7)
- added U205: NCP51460SN33T1G, Package_TO_SOT_SMD:SOT-23, F.Cu at (183.2, 66.5)
- C213, Q201, R202: moved to B.Cu
- D201: value MBR140SFT1G -> CRH01; footprint Diode_SMD:D_SOD-123F -> qdrive_footprints:SODFL3516X108N; moved to B.Cu
- J201: footprint qdrive_footprints:USB412003C -> qdrive_footprints:MOLEX_105450-0101
- R235: value 0R -> 0R/NC
- SW201: footprint qdrive_footprints:SW-SMD-4P -> qdrive_footprints:2192MST
- moved C211 10.3 mm to (200.1, 77.2), turned to 90 degrees
- moved R201 9.31 mm to (191.7, 52.5), turned to 90 degrees
- moved R233 8.54 mm to (180.2, 57.8)
- moved D201 7.95 mm to (199.8, 75.4)
- moved R230 7.91 mm to (205.5, 80.7)
- moved R205 7.91 mm to (203.9, 80.7)
- moved R203 7.90 mm to (202.3, 80.7)
- moved R207 7.55 mm to (202.5, 71.2)
- moved R208 7.51 mm to (204.8, 71.2)
- moved U203 7.42 mm to (203.3, 76.0)
- moved R229 7.00 mm to (184.2, 62.3)
- moved D203 6.96 mm to (191.0, 58.4)
- moved R227 6.80 mm to (200.7, 80.7)
- moved Q202 6.68 mm to (198.1, 66.9), turned to 90 degrees
- moved C212 6.58 mm to (186.7, 65.5)
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Routing:
- net GND: track 7.60 -> 41.4 mm, vias 165 -> 188
- net Net-(U205-Vout): track 0.00 -> 27.6 mm, vias 0 -> 2
- net +5VA: track 95.4 -> 119.2 mm, vias 3 -> 4
- net /main_board/M0_TEMP: track 49.3 -> 33.5 mm
- net +3V3: track 185.7 -> 172.5 mm, vias 12 -> 14
- net PGND_M0: track 2.82 -> 14.1 mm, vias 246 -> 238
- net /main_board/M1_CL: track 43.5 -> 33.6 mm
- net Net-(R229-Pad1): track 7.53 -> 15.7 mm
- net /main_board/M1_TEMP: track 34.8 -> 26.7 mm
- net /M0_board/M0_SP2: track 25.2 -> 17.1 mm
- net /main_board/CAN1_H: track 19.8 -> 27.1 mm, vias 0 -> 1
- net /M0_board/M0_GL_C: track 52.1 -> 44.8 mm
- net /main_board/AUX_N: track 24.3 -> 17.2 mm
- net /main_board/VDD_M: track 38.2 -> 31.5 mm
- net /main_board/AUX_P: track 22.4 -> 15.8 mm
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- added copper zone on In1.Cu, net /main_board/BRAKE_OUT
- added copper zone on In2.Cu, net /main_board/BRAKE_OUT
- added copper zone on B.Cu, net Net-(D201-K)
- added copper zone on F.Cu, net Net-(D201-K)
- added copper zone on In1.Cu, net PGND_MB
- added copper zone on In2.Cu, net PGND_MB
Other:
- board text added: "CAN GND H L"
- board text added: "CAN TERMINATION"
- board text added: "NC"
- board text added: "QDRIVE REV4 20230708"
- board text removed: "CAN H/L"
- board text removed: "CAN R"
- board text removed: "QDRIVE REV3 20230625"
