File: qmd_hw.kicad_pcb (KiCad board)
At the start: 4 copper layers, 60 x 175 mm, 267 parts, among them J201 USB4120-03-C, J203 Screw_Terminal_01x02, J204 X4621FVS-2x20-C43D65, J205 X4621WVS-2x20I-C40D64, J206 X4621FVS-2x20-C43D65, J207 X4621FVS-2x20-C43D65, J208 NC_Conn_02x03_Odd_Even, J209 JST_PH_B3B-PH-SM4-TB, J210 NC_Conn_01x07_Female, J211 S3B-PH-SM4-TB(LF)(SN)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

Commit message: Few updates
Parts:
- added REF**: WEEE-Logo_4.2x6mm_SilkScreen, Symbol:WEEE-Logo_4.2x6mm_SilkScreen, F.Cu at (210.9, 118.0)
Other:
- board text added: "https://github.com/kyuhyong/qmd_hw"
