File: M0_board.kicad_sch (KiCad schematic)
At the start: 88 parts, among them J301 Screw_Terminal_01x01, J302 Screw_Terminal_01x01, J303 Conn_01x05_MountingPin, J304 X4621WVS-2x20I-C40D64, J305 X4621FVS-2x20-C43D65, J306 Screw_Terminal_01x01, J307 Screw_Terminal_01x01, J309 Screw_Terminal_01x01, Q301 HYG025N06LS1C2, Q302 HYG025N06LS1C2, Q303 HYG025N06LS1C2, Q304 HYG025N06LS1C2, Q305 HYG025N06LS1C2, Q306 HYG025N06LS1C2, Q307 HYG025N06LS1C2, Q308 HYG025N06LS1C2, Q309 HYG025N06LS1C2, Q310 HYG025N06LS1C2, Q311 HYG025N06LS1C2, Q312 HYG025N06LS1C2, U301 DRV8301DCAR

Commit message: Update artwork for M0 board
Parts:
- removed NT303: NetTie_2, qdrive_footprints:NetTie-2_SMD_Pad2.0mm, symbol Device:NetTie_2
- added NT303: Net-Tie_2, NetTie:NetTie-2_SMD_Pad0.5mm, symbol bldc_motor_cntroller-rescue:Net-Tie_2-Device
Connections:
- net 3V3A: now also C336.1, U301.24 (REF)
- net GND1: now also C301.2, C304.2, C308.2, C314.2, C319.2, C322.2, C325.2, C327.2, C328.2, C329.2, C330.2, C331.2, C332.2, J305.10 (Pin_10), J305.12 (Pin_12), J305.14 (Pin_14), J305.16 (Pin_16), J305.18 (Pin_18), J305.20 (Pin_20), J305.22 (Pin_22), J305.24 (Pin_24), J305.26 (Pin_26), J305.28 (Pin_28), J305.30 (Pin_30), J305.32 (Pin_32), J305.34 (Pin_34), J305.36 (Pin_36), J305.38 (Pin_38), J305.4 (Pin_4), J305.40 (Pin_40), J305.6 (Pin_6), J305.8 (Pin_8), J309.1 (Pin_1), NT301.2, NT302.2, Q303.1 (S), Q303.2 (S), Q303.3 (S), Q304.1 (S), Q304.2 (S), Q304.3 (S), R312.1, R316.1, NT303.2
- removed net M0_3V3A: C336.1, J304.33 (Pin_33), U301.24 (REF)
- removed net PGND_M0: C301.2, C304.2, C308.2, C314.2, C319.2, C322.2, C325.2, C327.2, C328.2, C329.2, C330.2, C331.2, C332.2, J305.10 (Pin_10), J305.12 (Pin_12), J305.14 (Pin_14), J305.16 (Pin_16), J305.18 (Pin_18), J305.20 (Pin_20), J305.22 (Pin_22), J305.24 (Pin_24), J305.26 (Pin_26), J305.28 (Pin_28), J305.30 (Pin_30), J305.32 (Pin_32), J305.34 (Pin_34), J305.36 (Pin_36), J305.38 (Pin_38), J305.4 (Pin_4), J305.40 (Pin_40), J305.6 (Pin_6), J305.8 (Pin_8), J309.1 (Pin_1), NT301.2, NT302.2, Q303.1 (S), Q303.2 (S), Q303.3 (S), Q304.1 (S), Q304.2 (S), Q304.3 (S), R312.1, R316.1, U301.44 (SL_A)
- new net M0_SL_A: NT303.1, U301.44 (SL_A)
Other:
- moved on the sheet: C327, C328, C329, C330, C331, C332, C336, J302, J309

Commit message: Updated route per BOOSTXL reference design
Parts:
- removed TP301, TP302: TestPoint, TestPoint:TestPoint_Pad_D1.5mm, symbol Connector:TestPoint
- C307: footprint Capacitor_SMD:C_0402_1005Metric -> Capacitor_SMD:C_0603_1608Metric; JLCPN C159814 -> C57895; MPN CL05A225MA5NUNC -> CL10A225KA8NNNC
Other:
- note removed: "10K?"
Changed lines of the file:
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@@
-    (effects (font (size 1.27 1.27)) (justify left bottom))
-  )
-  (text "10K?" (at 92.71 68.58 0)
     (effects (font (size 1.27 1.27)) (justify left bottom))
   )
@@
         (path "/56ef7599-fa23-40e9-9d2c-9c83f71fd33c/c46210d2-0e3e-4934-a02e-e3590ff19e8b"
           (reference "Q303") (unit 1)
-        )
-      )
-    )
-  )
-  (symbol (lib_id "Connector:TestPoint") (at 184.15 139.7 0) (unit 1)
-    (in_bom yes) (on_board yes) (dnp no)
-    (property "Reference" "TP301" (at 185.6232 137.8712 0)
-      (effects (font (size 1.27 1.27)) (justify left))
-    )
-    (property "Value" "TestPoint" (at 185.6232 139.0142 0)
-      (effects (font (size 1.27 1.27)) (justify left) hide)
-    )
-    (property "Footprint" "TestPoint:TestPoint_Pad_D1.5mm" (at 189.23 139.7 0)
-      (effects (font (size 1.27 1.27)) hide)
-    )
-    (property "Datasheet" "~" (at 189.23 139.7 0)
-      (effects (font (size 1.27 1.27)) hide)
-    )
-    (property "MPN" "-" (at 184.15 139.7 0)
-      (effects (font (size 1.27 1.27)) hide)
-    )
-    (pin "1")
-    (instances
-      (project "qmd_hw"
-        (path "/56ef7599-fa23-40e9-9d2c-9c83f71fd33c/c46210d2-0e3e-4934-a02e-e3590ff19e8b"
-          (reference "TP301") (unit 1)
         )
       )
@@
       (effects (font (size 1.27 1.27)) (justify left))
     )
-    (property "Footprint" "Capacitor_SMD:C_0402_1005Metric" (at 175.26 52.07 0)
+    (property "Footprint" "Capacitor_SMD:C_0603_1608Metric" (at 175.26 52.07 0)
       (effects (font (size 1.27 1.27)) hide)
     )
@@
       (effects (font (size 1.27 1.27)) hide)
     )
-    (property "MPN" "CL05A225MA5NUNC" (at 175.26 52.07 0)
-      (effects (font (size 1.27 1.27)) hide)
-    )
-    (property "JLCPN" "C159814" (at 175.26 52.07 90)
+    (property "MPN" "CL10A225KA8NNNC" (at 175.26 52.07 0)
+      (effects (font (size 1.27 1.27)) hide)
+    )
+    (property "JLCPN" "C57895" (at 175.26 52.07 90)
       (effects (font (size 1.27 1.27)) hide)
     )
@@
         )
       )
-    )
-  )
-  (symbol (lib_id "Connector:TestPoint") (at 187.96 154.94 0) (unit 1)
-    (in_bom yes) (on_board yes) (dnp no)
-    (property "Reference" "TP302" (at 189.4332 153.1112 0)
-      (effects (font (size 1.27 1.27)) (justify left))
-    )
-    (property "Value" "TestPoint" (at 189.4332 154.2542 0)
-      (effects (font (size 1.27 1.27)) (justify left) hide)
-    )
-    (property "Footprint" "TestPoint:TestPoint_Pad_D1.5mm" (at 193.04 154.94 0)
-      (effects (font (size 1.27 1.27)) hide)
-    )
-    (property "Datasheet" "~" (at 193.04 154.94 0)
-      (effects (font (size 1.27 1.27)) hide)
-    )
-    (property "MPN" "-" (at 187.96 154.94 0)
-      (effects (font (size 1.27 1.27)) hide)
-    )
-    (pin "1")
-    (instances
-      (project "qmd_hw"
-        (path "/56ef7599-fa23-40e9-9d2c-9c83f71fd33c/c46210d2-0e3e-4934-a02e-e3590ff19e8b"
-          (reference "TP302") (unit 1)
-        )
-      )

Commit message: Fixed bugs and parts update
Parts:
- C311, C312, C323, C324: footprint Capacitor_SMD:C_0402_1005Metric -> Capacitor_SMD:C_0603_1608Metric
- C313, C316, C317, C318, C336: JLCPN C77020 -> (none); MPN GRM155R71H104KE14D -> (none)
- C326: footprint Capacitor_SMD:C_0402_1005Metric -> Capacitor_SMD:C_0603_1608Metric; JLCPN (none) -> C377773; MPN GRM155C81E225KE11D -> CL21A225KBQNNNE
- C333, C334, C335: footprint Capacitor_SMD:C_0402_1005Metric -> Capacitor_SMD:C_0603_1608Metric; JLCPN C77020 -> C1591; MPN GRM155R71H104KE14D -> CL10B104KB8NNNC
- R301, R302, R310, R311, R313, R314: footprint Resistor_SMD:R_0402_1005Metric -> Resistor_SMD:R_0603_1608Metric; JLCPN (none) -> C98220; MPN CRCW04022R20FKEDC -> RC0603FR-072R2L
- R307, R323: footprint Resistor_SMD:R_0402_1005Metric -> Resistor_SMD:R_0603_1608Metric; JLCPN (none) -> C114432; MPN CRCW04023K30FKEDC -> RC0603JR-073K3L
- R309, R315: footprint Resistor_SMD:R_0402_1005Metric -> Resistor_SMD:R_0603_1608Metric
- R319, R320, R321: footprint Resistor_SMD:R_0402_1005Metric -> Resistor_SMD:R_0603_1608Metric; MPN CRCW040210K0FKEDC -> RC0603FR-0710KL

Commit message: Updated MB
Parts:
- C307: JLCPN C57895 -> C913904; MPN CL10A225KA8NNNC -> CL10A225KB8NNNC
- C326: JLCPN C377773 -> C913904; MPN CL21A225KBQNNNE -> CL10A225KB8NNNC
Changed lines of the file:
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@@
       (effects (font (size 1.27 1.27)) hide)
     )
-    (property "MPN" "CL10A225KA8NNNC" (at 175.26 52.07 0)
-      (effects (font (size 1.27 1.27)) hide)
-    )
-    (property "JLCPN" "C57895" (at 175.26 52.07 90)
+    (property "MPN" "CL10A225KB8NNNC" (at 175.26 52.07 0)
+      (effects (font (size 1.27 1.27)) hide)
+    )
+    (property "JLCPN" "C913904" (at 175.26 52.07 90)
       (effects (font (size 1.27 1.27)) hide)
     )
@@
       (effects (font (size 1.27 1.27)) hide)
     )
-    (property "MPN" "CL21A225KBQNNNE" (at 254 97.79 0)
-      (effects (font (size 1.27 1.27)) hide)
-    )
-    (property "JLCPN" "C377773" (at 254 97.79 0)
-      (effects (font (size 1.27 1.27)) hide)
-    )
+    (property "MPN" "CL10A225KB8NNNC" (at 254 97.79 0)
+      (effects (font (size 1.27 1.27)) hide)
+    )
+    (property "JLCPN" "C913904" (at 254 97.79 0)
+      (effects (font (size 1.27 1.27)) hide)
+    )
