File: M1_board.kicad_sch (KiCad schematic)
At the start: 85 parts, among them J401 Screw_Terminal_01x01, J402 Screw_Terminal_01x01, J403 Screw_Terminal_01x01, J404 X4621WVS-2x20I-C40D64, J405 Screw_Terminal_01x01, J406 Conn_01x05_MountingPin, J408 X4621WVS-2x20I-C40D64, J409 Screw_Terminal_01x01, Q401 HYG025N06LS1C2, Q402 HYG025N06LS1C2, Q403 HYG025N06LS1C2, Q404 HYG025N06LS1C2, Q405 HYG025N06LS1C2, Q406 HYG025N06LS1C2, Q407 HYG025N06LS1C2, Q408 HYG025N06LS1C2, Q409 HYG025N06LS1C2, Q410 HYG025N06LS1C2, Q411 HYG025N06LS1C2, Q412 HYG025N06LS1C2, U401 DRV8301DCAR

Commit message: Fixed bugs and parts update
Parts:
- removed NT403: NetTie_2, qdrive_footprints:NetTie-2_SMD_Pad2.0mm, symbol Device:NetTie_2
- removed TP401, TP402: TestPoint, TestPoint:TestPoint_Pad_D1.5mm, symbol Connector:TestPoint
- added C434: 0.1uF 50V, Capacitor_SMD:C_0402_1005Metric, symbol Device:C_Small
- added NT404: Net-Tie_2, NetTie:NetTie-2_SMD_Pad0.5mm, symbol bldc_motor_cntroller-rescue:Net-Tie_2-Device
- C407, C423: footprint Capacitor_SMD:C_0402_1005Metric -> Capacitor_SMD:C_0603_1608Metric; JLCPN C159814 -> C377773; MPN CL05A225MA5NUNC -> CL21A225KBQNNNE
- C411, C412, C421: footprint Capacitor_SMD:C_0402_1005Metric -> Capacitor_SMD:C_0603_1608Metric
- C413, C415, C416, C417: JLCPN C77020 -> (none); MPN GRM155R71H104KE14D -> (none)
- C424, C425, C426, C433: footprint Capacitor_SMD:C_0402_1005Metric -> Capacitor_SMD:C_0603_1608Metric; JLCPN C77020 -> C1591; MPN GRM155R71H104KE14D -> CL10B104KB8NNNC
- R401, R402, R410, R411, R413, R414: footprint Resistor_SMD:R_0402_1005Metric -> Resistor_SMD:R_0603_1608Metric; JLCPN (none) -> C98220; MPN CRCW04022R20FKEDC -> RC0603FR-072R2L
- R407, R423: footprint Resistor_SMD:R_0402_1005Metric -> Resistor_SMD:R_0603_1608Metric; JLCPN (none) -> C114432; MPN CRCW04023K30FKEDC -> RC0603JR-073K3L
- R409, R415: footprint Resistor_SMD:R_0402_1005Metric -> Resistor_SMD:R_0603_1608Metric
- R419, R420, R421: footprint Resistor_SMD:R_0402_1005Metric -> Resistor_SMD:R_0603_1608Metric; MPN CRCW040210K0FKEDC -> RC0603FR-0710KL
Connections:
- net 3V3B: now also C433.1, U401.24 (REF), C434.1
- net GND2: now also C401.2, C404.2, C408.2, C414.2, C418.2, C420.2, C422.2, C427.2, C428.2, C429.2, C430.2, C431.2, C432.2, J408.10 (Pin_10), J408.12 (Pin_12), J408.14 (Pin_14), J408.16 (Pin_16), J408.18 (Pin_18), J408.20 (Pin_20), J408.22 (Pin_22), J408.24 (Pin_24), J408.26 (Pin_26), J408.28 (Pin_28), J408.30 (Pin_30), J408.32 (Pin_32), J408.34 (Pin_34), J408.36 (Pin_36), J408.38 (Pin_38), J408.4 (Pin_4), J408.40 (Pin_40), J408.6 (Pin_6), J408.8 (Pin_8), J409.1 (Pin_1), NT401.2, NT402.2, Q403.1 (S), Q403.2 (S), Q403.3 (S), Q404.1 (S), Q404.2 (S), Q404.3 (S), R412.1, R416.1, C434.2, NT404.2
- net M1_3V3A: no longer C433.1, U401.24 (REF)
- removed net PGND_M1: C401.2, C404.2, C408.2, C414.2, C418.2, C420.2, C422.2, C427.2, C428.2, C429.2, C430.2, C431.2, C432.2, J408.10 (Pin_10), J408.12 (Pin_12), J408.14 (Pin_14), J408.16 (Pin_16), J408.18 (Pin_18), J408.20 (Pin_20), J408.22 (Pin_22), J408.24 (Pin_24), J408.26 (Pin_26), J408.28 (Pin_28), J408.30 (Pin_30), J408.32 (Pin_32), J408.34 (Pin_34), J408.36 (Pin_36), J408.38 (Pin_38), J408.4 (Pin_4), J408.40 (Pin_40), J408.6 (Pin_6), J408.8 (Pin_8), J409.1 (Pin_1), NT401.2, NT402.2, Q403.1 (S), Q403.2 (S), Q403.3 (S), Q404.1 (S), Q404.2 (S), Q404.3 (S), R412.1, R416.1, U401.44 (SL_A)
- new net M1_SL_A: NT404.1, U401.44 (SL_A)
Other:
- moved on the sheet: C433, R404

Commit message: Updated MB
Parts:
- C407, C423: JLCPN C377773 -> C913904; MPN CL21A225KBQNNNE -> CL10A225KB8NNNC
Changed lines of the file:
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@@
       (effects (font (size 1.27 1.27)) hide)
     )
-    (property "MPN" "CL21A225KBQNNNE" (at 240.03 99.06 0)
-      (effects (font (size 1.27 1.27)) hide)
-    )
-    (property "JLCPN" "C377773" (at 240.03 99.06 90)
+    (property "MPN" "CL10A225KB8NNNC" (at 240.03 99.06 0)
+      (effects (font (size 1.27 1.27)) hide)
+    )
+    (property "JLCPN" "C913904" (at 240.03 99.06 90)
       (effects (font (size 1.27 1.27)) hide)
     )
@@
       (effects (font (size 1.27 1.27)) hide)
     )
-    (property "MPN" "CL21A225KBQNNNE" (at 161.29 53.34 0)
-      (effects (font (size 1.27 1.27)) hide)
-    )
-    (property "JLCPN" "C377773" (at 161.29 53.34 90)
-      (effects (font (size 1.27 1.27)) hide)
-    )
+    (property "MPN" "CL10A225KB8NNNC" (at 161.29 53.34 0)
+      (effects (font (size 1.27 1.27)) hide)
+    )
+    (property "JLCPN" "C913904" (at 161.29 53.34 90)
+      (effects (font (size 1.27 1.27)) hide)
+    )
