File: main_board.kicad_sch (KiCad schematic)
At the start: 91 parts, among them J201 USB4120-03-C, J202 B2B-PH-SM4-TB(LF)(SN), J203 Screw_Terminal_01x02, J204 X4621FVS-2x20-C43D65, J205 X4621WVS-2x20I-C40D64, J206 X4621FVS-2x20-C43D65, J207 X4621FVS-2x20-C43D65, J208 NC_Conn_02x03_Odd_Even, J209 JST_PH_B3B-PH-SM4-TB, J210 NC_Conn_01x07_Female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

Commit message: Fixed bugs and parts update
Parts:
- removed C221: 4.7uF 50V, Capacitor_SMD:C_0805_2012Metric, symbol Device:C_Small
- removed U205: LP5907MFX-3.3, Package_TO_SOT_SMD:SOT-23-5, symbol Regulator_Linear:LP5907MFX-3.3
- added R235: 0R, Resistor_SMD:R_0603_1608Metric, symbol Device:R_Small
- C201, C205, C211: footprint Capacitor_SMD:C_0402_1005Metric -> Capacitor_SMD:C_0603_1608Metric; JLCPN C159814 -> C377773; MPN CL05A225MA5NUNC -> CL21A225KBQNNNE
- C202, C203, C204, C206, C207, C210, C212, C213, C217: footprint Capacitor_SMD:C_0402_1005Metric -> Capacitor_SMD:C_0603_1608Metric; JLCPN C77020 -> C1591; MPN GRM155R71H104KE14D -> CL10B104KB8NNNC
- C208, C209, C214, C215, C216, C218, C219, C223, C224, C225, C226: footprint Capacitor_SMD:C_0402_1005Metric -> Capacitor_SMD:C_0603_1608Metric
- R201, R212, R213, R214, R215, R216, R217, R222, R223, R224, R225, R227, R230, R231, R232: footprint Resistor_SMD:R_0402_1005Metric -> Resistor_SMD:R_0603_1608Metric; JLCPN (none) -> C114432; MPN CRCW04023K30FKEDC -> RC0603JR-073K3L
- R202, R226, R233, R234: footprint Resistor_SMD:R_0402_1005Metric -> Resistor_SMD:R_0603_1608Metric
- R203: footprint Resistor_SMD:R_0402_1005Metric -> Resistor_SMD:R_0603_1608Metric; JLCPN C4105840 -> C95177; MPN ERJ-H2G0R00X -> RC0603JR-070RL
- R204: footprint Resistor_SMD:R_0402_1005Metric -> Resistor_SMD:R_0603_1608Metric; MPN CRCW040210K0FKEDC -> RC0603FR-0710KL
- R205, R206, R211, R218, R219, R220, R221, R228, R229: footprint Resistor_SMD:R_0402_1005Metric -> Resistor_SMD:R_0603_1608Metric; JLCPN (none) -> C95177; MPN (none) -> RC0603JR-070RL
- R207, R208: footprint Resistor_SMD:R_0402_1005Metric -> Resistor_SMD:R_0603_1608Metric; JLCPN (none) -> C98220; MPN CRCW04022R20FKEDC -> RC0603FR-072R2L
- R209: footprint Resistor_SMD:R_0402_1005Metric -> Resistor_SMD:R_0603_1608Metric; JLCPN (none) -> C112307
- R210: footprint Resistor_SMD:R_0402_1005Metric -> Resistor_SMD:R_0603_1608Metric; JLCPN (none) -> C513397; MPN ERJ-2RKF1001X -> RT0603BRE071KL
Connections:
- net +3.3VA: now also R235.2
- net +3V3: now also R235.1

Commit message: Updated MB
Parts:
- removed J202: B2B-PH-SM4-TB(LF)(SN), Connector_JST:JST_PH_B2B-PH-SM4-TB_1x02-1MP_P2.00mm_Vertical, symbol Connector_Generic_MountingPin:Conn_01x02_MountingPin
- added C221: 0.1uF 50V, Capacitor_SMD:C_0603_1608Metric, symbol Device:C_Small
- added C227: 1uF 35V, Capacitor_SMD:C_0603_1608Metric, symbol Device:C_Small
- added J211: S3B-PH-SM4-TB(LF)(SN), qdrive_footprints:JST_S3B-PH-SM4-TB, symbol Connector_Generic_MountingPin:Conn_01x03_MountingPin
- added JP207: Jumper_2_Open, Jumper:SolderJumper-2_P1.3mm_Open_TrianglePad1.0x1.5mm, symbol Jumper:Jumper_2_Open
- added Q203, Q204: CSD18540Q5B, Package_TO_SOT_SMD:TDSON-8-1, symbol Transistor_FET:CSD18540Q5B
- added R236: 0R, Resistor_SMD:R_0603_1608Metric, symbol Device:R_Small
- added U205: NCP51460SN33T1G, Package_TO_SOT_SMD:SOT-23, symbol Reference_Voltage:MCP1525-TT
- C201, C205, C211: JLCPN C377773 -> C913904; MPN CL21A225KBQNNNE -> CL10A225KB8NNNC
- D201: value MBR140SFT1G -> CRH01; footprint Diode_SMD:D_SOD-123F -> qdrive_footprints:SODFL3516X108N; JLCPN C193342 -> C845528; MPN PMEG4010CEH,115 -> CRH01(TE85L,Q)
- R207, R208: JLCPN C98220 -> C112307
- R235: value 0R -> 0R/NC
Connections:
- net +3.3VA: now also R236.2
- net +48V: now also Q204.5 (D)
- net +5VA: now also C221.2, JP207.2 (B), U205.1 (Vin)
- net BRAKE_OUT: now also Q203.5 (D), Q204.1 (S), Q204.2 (S), Q204.3 (S)
- net CAN1_H: now also J211.2 (Pin_2)
- net CAN1_L: now also J211.3 (Pin_3)
- net GND: now also C221.1, C227.2, J211.1 (Pin_1), J211.MP (MountPin), U205.3 (Vss)
- net PGND_MB: now also Q203.1 (S), Q203.2 (S), Q203.3 (S)
- net USB_V: now also JP207.1 (A)
- net at Q201.4 (G), R207.2: now also Q204.4 (G)
- net at Q202.4 (G), R208.2: now also Q203.4 (G)
- new net: C227.1, R236.1, U205.2 (Vout)
